File: 180V_power/tube_power.brd (EAGLE design)
At the start: 55 x 30 mm, 28 parts, among them IC1 NE555D, Q1 IRF740S, U1 TLV1117-5SOT-223, U2 BC817

Commit message: fixed document info
Parts:
- U2: value BC817 -> 2N7002
