File: 180V_power/tube_power.brd (EAGLE design)
At the start: 55 x 30 mm, 28 parts, among them IC1 NE555D, Q1 IRF740S, U1 TLV1117-5SOT-223, U2 2N7002

Commit message: update document data
Parts:
- C4: value 2.2uF -> 10uF
- R2: value (none) -> 1K
- U2: value 2N7002 -> BC817
Other:
- board text added: "D2"
